Commit message: Add cooperative multi-agent tasks: pushball, pushbox, gate_with_button
Add three new cooperative multi-agent tasks for Go1 quadruped robots.

  - pushball: agents cooperate to push a ball to the target zone
  - pushbox: agents cooperate to push a box (light/medium variants)
  - gate_with_button: one agent presses button to open gate while others pass through

  Includes configs, wrappers, URDF assets, and verification scripts for each task.

File: resources/objects/ball_heavy.urdf (robot description, URDF)
Before this commit: robot ball, 1 links, 0 joints
Links:
- removed link ball
- added link ball_heavy, mass 10.0; collision sphere radius=0.5; visual sphere radius=0.5

File: resources/objects/ball_large.urdf (robot description, URDF)
Before this commit: robot ball, 1 links, 0 joints
Links:
- removed link ball
- added link ball_large, mass 3.0; collision sphere radius=0.5; visual sphere radius=0.5

File: resources/objects/box_light.urdf (robot description, URDF)
Before this commit: robot ball, 1 links, 0 joints
Links:
- removed link ball
- added link box, mass 1; collision box size=1 1 1; visual box size=1 1 1

File: resources/objects/box_medium.urdf (robot description, URDF)
Before this commit: robot ball, 1 links, 0 joints
Links:
- removed link ball
- added link box, mass 3; collision box size=1 1 1; visual box size=1 1 1
